File: DRV8313_Dev_Board_Hardware/DRV8313_Dev_Board.kicad_pcb (KiCad board)
At the start: 2 copper layers, 7 parts, among them IC1 DRV8313PWP, IC2 INA199A1DCKR, IC3 INA199A1DCKR, IC4 INA199A1DCKR, IC5 STM32F103C8T6TR, Y1 32.768KHZ_YST310S

Commit message: Updata SCH Alpha0.2
Parts:
- added C10: 4.7uF, Capacitor_SMD:C_0603_1608Metric, F.Cu at (20.4, 24.7)
- added C11: 0.1uF, Capacitor_SMD:C_0603_1608Metric, F.Cu at (20.4, 27.2)
- added C12: 2.2uF, Capacitor_SMD:C_0603_1608Metric, F.Cu at (20.4, 29.7)
- added C13: 4.7uF, Capacitor_SMD:C_0603_1608Metric, F.Cu at (24.4, 22.2)
- added C14: 0.1uF, Capacitor_SMD:C_0603_1608Metric, F.Cu at (24.4, 24.7)
- added C15: 1uF, Capacitor_SMD:C_0603_1608Metric, F.Cu at (24.4, 27.2)
- added C16: 1uF, Capacitor_SMD:C_0603_1608Metric, F.Cu at (24.4, 29.7)
- added C9: 4.7uF, Capacitor_SMD:C_0603_1608Metric, F.Cu at (20.4, 22.2)
- added IC6: XC6206P332MR, SamacSys_Parts:SOT95P240X115-3N, F.Cu at (32.8, 23.2)
- added J2: Connector_Pin, Connector_PinHeader_2.54mm:PinHeader_1x04_P2.54mm_Vertical, F.Cu at (16.0, 23.3)
- added R5: 4.7K, Resistor_SMD:R_0603_1608Metric, F.Cu at (28.4, 22.2)
- added R6: 4.7K, Resistor_SMD:R_0603_1608Metric, F.Cu at (28.4, 24.7)
- added R7: 4.7K, Resistor_SMD:R_0603_1608Metric, F.Cu at (28.4, 27.2)
- added R8: 560K, Resistor_SMD:R_0603_1608Metric, F.Cu at (28.4, 29.7)
- added U1: 中景园_0.87寸OLED, kicad_lceda:中景园0.87寸OLED, F.Cu at (38.9, 15.9)
- added Y2: YSX321SL, SamacSys_Parts:YSX321SL, F.Cu at (35.8, 36.1)
Connections:
- IC5 pad 1: unconnected-(IC5-VBAT-Pad1) -> +3.3V
- IC5 pad 13: unconnected-(IC5-PA3-Pad13) -> /VSENSE_DC_IN
- IC5 pad 24: unconnected-(IC5-VDD_1-Pad24) -> +3.3V
- IC5 pad 26: unconnected-(IC5-PB13-Pad26) -> /EN1
- IC5 pad 27: unconnected-(IC5-PB14-Pad27) -> /EN2
- IC5 pad 28: unconnected-(IC5-PB15-Pad28) -> /EN3
- IC5 pad 36: unconnected-(IC5-VDD_2-Pad36) -> +3.3V
- IC5 pad 39: unconnected-(IC5-PB3-Pad39) -> /FAULT
- IC5 pad 40: unconnected-(IC5-PB4-Pad40) -> /SLEEP
- IC5 pad 41: unconnected-(IC5-PB5-Pad41) -> /RESET
- IC5 pad 48: unconnected-(IC5-VDD_3-Pad48) -> +3.3V
- IC5 pad 5: unconnected-(IC5-PD0-OSC_IN-Pad5) -> /OSC_IN
- IC5 pad 6: unconnected-(IC5-PD1-OSC_OUT-Pad6) -> /OSC_OUT
- IC5 pad 9: unconnected-(IC5-VDDA-Pad9) -> +3.3V

Commit message: Updata SCH Alpha0.3
Parts:
- added C1: 0.1uF, Capacitor_SMD:C_0603_1608Metric, F.Cu at (23.1, 60.6)
- added C17: 4.7uF, Capacitor_SMD:C_0603_1608Metric, F.Cu at (48.4, 150.1)
- added C18: 470uF, Capacitor_SMD:CP_Elec_6.3x5.7, F.Cu at (85.1, 73.9)
- added C19: 1uF, Capacitor_SMD:C_0603_1608Metric, F.Cu at (27.1, 78.2)
- added C2: 1uF, Capacitor_SMD:C_0603_1608Metric, F.Cu at (23.1, 63.1)
- added C20: 0.01uF, Capacitor_SMD:C_0603_1608Metric, F.Cu at (27.1, 80.7)
- added C21: 4.7uF, Capacitor_SMD:C_0603_1608Metric, F.Cu at (27.1, 83.2)
- added C22: 4.7uF, Capacitor_SMD:C_0603_1608Metric, F.Cu at (31.1, 60.6)
- added C23: 0.1uF, Capacitor_SMD:C_0603_1608Metric, F.Cu at (31.1, 63.1)
- added C24: 2.2uF, Capacitor_SMD:C_0603_1608Metric, F.Cu at (31.1, 65.6)
- added C25: 4.7uF, Capacitor_SMD:C_0603_1608Metric, F.Cu at (31.1, 68.2)
- added C26: 0.1uF, Capacitor_SMD:C_0603_1608Metric, F.Cu at (31.1, 70.7)
- added C27: 1uF, Capacitor_SMD:C_0603_1608Metric, F.Cu at (31.1, 73.2)
- added C28: 1uF, Capacitor_SMD:C_0603_1608Metric, F.Cu at (31.1, 75.7)
- added C3: 47pF, Capacitor_SMD:C_0603_1608Metric, F.Cu at (23.1, 65.6)
- added C30: 0.47uF, Capacitor_SMD:C_0603_1608Metric, F.Cu at (31.1, 78.2)
- added C31: 0.1uF, Capacitor_SMD:C_0603_1608Metric, F.Cu at (31.1, 80.7)
- added C32: 0.01uF/60V, Capacitor_SMD:C_0603_1608Metric, F.Cu at (31.1, 83.2)
- added C33: 0.1uF/16V, Capacitor_SMD:C_0603_1608Metric, F.Cu at (35.1, 60.6)
- added C4: 47pf, Capacitor_SMD:C_0603_1608Metric, F.Cu at (23.1, 68.2)
- added C5: 0.1uF, Capacitor_SMD:C_0603_1608Metric, F.Cu at (50.2, 163.2)
- added C6: 47pF, Capacitor_SMD:C_0603_1608Metric, F.Cu at (23.1, 73.2)
- added C7: 1uF, Capacitor_SMD:C_0603_1608Metric, F.Cu at (23.1, 75.7)
- added C8: 0.01uF, Capacitor_SMD:C_0603_1608Metric, F.Cu at (23.1, 78.2)
- added D1: SS54, SamacSys_Parts:DIOM5126X245N, F.Cu at (51.0, 153.2)
- added D3: 1N4148WS, Diode_SMD:D_SOD-323, F.Cu at (69.8, 55.0)
- added D4: SS54, SamacSys_Parts:DIOM5126X245N, F.Cu at (49.3, 158.3)
- added D5: FAULT, LED_SMD:LED_0603_1608Metric, F.Cu at (69.7, 57.8)
- added IC7: INA199A1DCKR, SamacSys_Parts:SOT65P210X110-6N, F.Cu at (78.5, 155.1)
- added IC8: DRV8313PWP, SamacSys_Parts:SOP65P640X120-29N, F.Cu at (74.1, 148.5)
- added J1: HALL_Sensor_Port, Connector_JST:JST_GH_SM05B-GHS-TB_1x05-1MP_P1.25mm_Horizontal, F.Cu at (90.6, 172.9)
- added J3: AS5600_Port, Connector_JST:JST_GH_BM04B-GHS-TBT_1x04-1MP_P1.25mm_Vertical, F.Cu at (57.6, 173.4)
- added J4: USB_C_Receptacle, Connector_USB:USB_C_Receptacle_XKB_U262-16XN-4BVC11, F.Cu at (36.2, 133.3)
- added J5: CAN_BUS_Port_OUT, Connector_JST:JST_GH_BM02B-GHS-TBT_1x02-1MP_P1.25mm_Vertical, F.Cu at (108.2, 142.6)
- added J6: DC_IN, Connector_AMASS:AMASS_XT30PW-M_1x02_P2.50mm_Horizontal, F.Cu at (45.3, 148.2)
- added J7: DC_OUT, Connector_AMASS:AMASS_XT30PW-M_1x02_P2.50mm_Horizontal, F.Cu at (98.0, 155.8)
- added J8: Conn_01x03_Socket, Connector_AMASS:AMASS_MR30PW-M_1x03_P3.50mm_Horizontal, F.Cu at (77.6, 162.9)
- added L1: 15uH, Inductor_SMD:L_Bourns-SRN4018, F.Cu at (59.3, 166.1)
- added R1: 10K, Resistor_SMD:R_0603_1608Metric, F.Cu at (35.1, 63.1)
- added R10: 4.7K, Resistor_SMD:R_0603_1608Metric, F.Cu at (39.1, 60.6)
- added R11: 5K1, Resistor_SMD:R_0603_1608Metric, F.Cu at (39.1, 63.1)
- added R12: 5K1, Resistor_SMD:R_0603_1608Metric, F.Cu at (39.1, 65.6)
- added R13: 4.99K, Resistor_SMD:R_0603_1608Metric, F.Cu at (39.1, 68.2)
- added R14: 500mR, Resistor_SMD:R_1206_3216Metric, F.Cu at (68.8, 158.8)
- added R15: 500mR, Resistor_SMD:R_1206_3216Metric, F.Cu at (73.9, 158.8)
- added R16: 500mR, Resistor_SMD:R_1206_3216Metric, F.Cu at (78.8, 158.7)
- added R17: 120R, Resistor_SMD:R_0603_1608Metric, F.Cu at (77.3, 101.2)
- added R18: 0R, Resistor_SMD:R_0603_1608Metric, F.Cu at (77.3, 99.8)
- added R2: 10K, Resistor_SMD:R_0603_1608Metric, F.Cu at (55.4, 163.2)
- added R3: 3.16K, Resistor_SMD:R_0603_1608Metric, F.Cu at (52.4, 163.2)
- added R4: 10K, Resistor_SMD:R_0603_1608Metric, F.Cu at (35.1, 70.7)
- added R9: 560K, Resistor_SMD:R_0603_1608Metric, F.Cu at (35.1, 83.2)
- added U2: 中景园_0.87寸OLED, kicad_lceda:中景园0.87寸OLED, F.Cu at (91.6, 132.9)
- added U3: SN65HVD232, Package_SO:SOIC-8_3.9x4.9mm_P1.27mm, F.Cu at (57.2, 144.4)
- C10, C13, C9: value 4.7uF -> 0.1uF
- C12: value 2.2uF -> 4.7uF
- C14: value 0.1uF -> 4.7uF
- C16: value 1uF -> 47pF
- IC1: value DRV8313PWP -> LP2992IM5-3.3; footprint SamacSys_Parts:SOP65P640X120-29N -> SamacSys_Parts:SOT95P280X145-5N
- IC2: value INA199A1DCKR -> STM32F103C8T6TR; footprint SamacSys_Parts:SOT65P210X110-6N -> SamacSys_Parts:QFP50P900X900X160-48N
- IC3: value INA199A1DCKR -> TPS5450DDAR; footprint SamacSys_Parts:SOT65P210X110-6N -> SamacSys_Parts:SOIC127P600X170-9N
- IC4: value INA199A1DCKR -> LP2992IM5-3.3; footprint SamacSys_Parts:SOT65P210X110-6N -> SamacSys_Parts:SOT95P280X145-5N
- IC5: value STM32F103C8T6TR -> INA199A1DCKR; footprint SamacSys_Parts:QFP50P900X900X160-48N -> SamacSys_Parts:SOT65P210X110-6N
- IC6: value XC6206P332MR -> INA199A1DCKR; footprint SamacSys_Parts:SOT95P240X115-3N -> SamacSys_Parts:SOT65P210X110-6N
- J2: value Connector_Pin -> CAN_BUS_Port_IN; footprint Connector_PinHeader_2.54mm:PinHeader_1x04_P2.54mm_Vertical -> Connector_JST:JST_GH_BM02B-GHS-TBT_1x02-1MP_P1.25mm_Vertical
- R8: value 560K -> 4.7K
- U1: value 中景园_0.87寸OLED -> CP2102N-Axx-xQFN28; footprint kicad_lceda:中景园0.87寸OLED -> Package_DFN_QFN:QFN-28-1EP_5x5mm_P0.5mm_EP3.35x3.35mm
- moved J2 145.0 mm to (99.5, 141.9), turned to -90 degrees
- moved IC6 138.1 mm to (73.6, 155.2), turned to -90 degrees
- moved IC3 124.7 mm to (53.7, 158.7), turned to 90 degrees
- moved C12 124.0 mm to (50.2, 150.1), turned to 90 degrees
- moved IC5 123.8 mm to (68.5, 155.2)
- moved D2 118.9 mm to (58.2, 158.6), turned to 90 degrees
- moved U1 117.5 mm to (46.5, 133.1)
- moved IC4 107.8 mm to (50.4, 145.7)
- moved IC2 103.9 mm to (57.6, 133.5), turned to -90 degrees
- moved IC1 96.8 mm to (50.4, 141.1), turned to 0 degrees
- moved Y2 82.9 mm to (73.9, 109.8), turned to -90 degrees
- moved Y1 69.3 mm to (73.9, 103.1), turned to 90 degrees
- moved C9 58.6 mm to (23.1, 80.7)
- moved C10 58.6 mm to (23.1, 83.2)
- moved R6 51.4 mm to (35.1, 75.7)
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Connections:
- C10 pad 1: GND -> +3.3V
- C10 pad 2: /VCC_OLED -> GND
- C11 pad 1: GND -> +3.3V
- C11 pad 2: /VCC_OLED -> GND
- C12 pad 1: GND -> VCC
- C12 pad 2: Net-(U1-VCOMH) -> GND
- C13 pad 1: GND -> +3.3V
- C13 pad 2: Net-(U1-VCC) -> GND
- C14 pad 1: GND -> +5V
- C14 pad 2: Net-(U1-VCC) -> GND
- C15 pad 1: Net-(U1-c2n) -> +5V
- C15 pad 2: Net-(U1-c2p) -> GND
- C16 pad 1: Net-(U1-c1n) -> GND
- C16 pad 2: Net-(U1-c1p) -> /OSC_OUT
- C9 pad 1: GND -> +3.3V
- C9 pad 2: Net-(U1-RES#) -> GND
- D2 pad 1: VCC -> Net-(D2-K)
- IC1 pad 1: Net-(IC1-CPL) -> +5V
- IC1 pad 2: Net-(IC1-CPH) -> GND
- IC1 pad 3: Net-(IC1-VCP) -> +5V
- IC1 pad 4: VCC -> Net-(IC1-BYPASS)
- IC1 pad 5: /OUT1 -> +3.3V
- IC2 pad 1: GND -> +3.3V
- IC2 pad 2: GND -> unconnected-(IC2-PC13-TAMPER-RT_C-Pad2)
- IC2 pad 3: /V3P3_OUT -> /OSC32_IN
- IC2 pad 4: /Motor0_U -> /OSC32_OUT
- IC2 pad 5: /OUT1 -> /OSC_IN
- IC2 pad 6: /ISense_U -> /OSC_OUT
- IC3 pad 1: GND -> Net-(IC3-BOOT)
- IC3 pad 2: GND -> unconnected-(IC3-NC_1-Pad2)
- IC3 pad 3: /V3P3_OUT -> unconnected-(IC3-NC_2-Pad3)
- IC3 pad 4: /Motor0_V -> Net-(IC3-VSENSE)
- IC3 pad 5: /OUT2 -> unconnected-(IC3-ENA-Pad5)
- IC3 pad 6: /ISense_V -> GND
- IC4 pad 1: GND -> +5V
- IC4 pad 3: /V3P3_OUT -> +5V
- IC4 pad 4: /Motor0_W -> Net-(IC4-BYPASS)
- IC4 pad 5: /OUT3 -> /VCC_Sensor
- IC5 pad 1: +3.3V -> GND
- IC5 pad 2: unconnected-(IC5-PC13-TAMPER-RT_C-Pad2) -> GND
- IC5 pad 3: /OSC32_IN -> /V3P3_OUT
- IC5 pad 4: /OSC32_OUT -> /Motor0_U
- IC5 pad 5: /OSC_IN -> /OUT1
- IC5 pad 6: /OSC_OUT -> /ISense_U
- IC6 pad 2: /VCC_OLED -> GND
- IC6 pad 3: /VCC_IN -> /V3P3_OUT
- J2 pad 1: GND -> /CAN_DP
- J2 pad 2: /VCC_IN -> /CAN_DN
- R7 pad 1: /VCC_OLED -> +3.3V
- R7 pad 2: Net-(U1-RES#) -> Net-(U2-RES#)
- R8 pad 1: GND -> +3.3V
- R8 pad 2: Net-(U1-IREF) -> /AS5600_SCL
- U1 pad 1: Net-(U1-c2p) -> unconnected-(U1-~{DCD}-Pad1)
- U1 pad 10: /OLED_SCL -> unconnected-(U1-NC-Pad10)
- U1 pad 11: /OLED_SDA -> unconnected-(U1-~{SUSPEND}-Pad11)
- U1 pad 12: Net-(U1-IREF) -> unconnected-(U1-SUSPEND-Pad12)
- U1 pad 13: Net-(U1-VCOMH) -> unconnected-(U1-CHREN-Pad13)
- U1 pad 14: Net-(U1-VCC) -> unconnected-(U1-CHR1-Pad14)
- U1 pad 2: Net-(U1-c2n) -> unconnected-(U1-~{RI}/CLK-Pad2)
- U1 pad 3: Net-(U1-c1p) -> GND
- U1 pad 4: Net-(U1-c1n) -> /USB_DP
- U1 pad 5: /VCC_OLED -> /USB_DN
- U1 pad 7: GND -> +5V
- U1 pad 8: /VCC_OLED -> +5V
- U1 pad 9: Net-(U1-RES#) -> Net-(U1-~{RST})
Other:
- board outline added: 80 x 48.6 mm
