File: DRV8313_Dev_Board_Hardware/DRV8313_Dev_Board.kicad_sch (KiCad schematic)
At the start: 19 parts, among them IC1 DRV8313PWP, IC2 INA199A1DCKR, IC3 INA199A1DCKR, IC4 INA199A1DCKR, IC5 STM32F103C8T6TR, J1 DC_IN, Y1 32.768KHZ_YST310S

Commit message: Updata SCH Alpha0.2
Parts:
- added C10, C13, C9: 4.7uF, Capacitor_SMD:C_0603_1608Metric, symbol oled:C
- added C11, C14: 0.1uF, Capacitor_SMD:C_0603_1608Metric, symbol oled:C
- added C12: 0.1uF, Capacitor_SMD:C_0603_1608Metric, symbol Device:C
- added C12: 2.2uF, Capacitor_SMD:C_0603_1608Metric, symbol oled:C
- added C15, C16: 1uF, Capacitor_SMD:C_0603_1608Metric, symbol oled:C
- added C17, C19: 1uF, symbol Device:C
- added C17, C18, C19: 4.7uF, Capacitor_SMD:C_0603_1608Metric, symbol Device:C
- added C18: 0.01uF, symbol Device:C
- added C20: 470uF, Capacitor_SMD:CP_Elec_6.3x5.7, symbol Device:C_Polarized
- added C25, C26, C27, C28, C29: 0.1uF, symbol Device:C
- added C7, C8: C, symbol Device:C
- added D3, D5: SS54, DIOM5126X245N, symbol SamacSys_Parts:SS54
- added D4: 1N4148WS, Diode_SMD:D_SOD-323, symbol Diode:1N4148WS
- added IC6: XC6206P332MR, SOT95P240X115-3N, symbol oled:XC6206P332MR
- added IC7: LP2992IM5-3.3, SOT95P280X145-5N, symbol SamacSys_Parts:LP2992IM5-3.3
- added IC8: TPS5450DDAR, SOIC127P600X170-9N, symbol SamacSys_Parts:TPS5450DDAR
- added J2: USB_C_Receptacle, symbol Connector:USB_C_Receptacle
- added L1: 15uH, Inductor_SMD:L_Bourns-SRN4018, symbol Device:L
- added R11, R15: 10K, symbol Device:R
- added R12, R13: 5K1, symbol Device:R
- added R34: 10K, Resistor_SMD:R_0603_1608Metric, symbol Device:R
- added R35: 3.16K, Resistor_SMD:R_0603_1608Metric, symbol Device:R
- added R5, R6, R7: 4.7K, Resistor_SMD:R_0603_1608Metric, symbol oled:R
- added R8: 560K, Resistor_SMD:R_0603_1608Metric, symbol oled:R
- added U1: 中景园_0.87寸OLED, kicad_lceda:中景园0.87寸OLED, symbol oled:中景园_0.87寸OLED
- added U2: SN65HVD232, Package_SO:SOIC-8_3.9x4.9mm_P1.27mm, symbol Interface_CAN_LIN:SN65HVD232
- added U3: CP2102N-Axx-xQFN28, Package_DFN_QFN:QFN-28-1EP_5x5mm_P0.5mm_EP3.35x3.35mm, symbol Interface_USB:CP2102N-Axx-xQFN28
- added Y2: YSX321SL, YSX321SL, symbol SamacSys_Parts:YSX321SL
Connections:
- net GND: now also IC5.23 (VSS_1), IC5.35 (VSS_2), IC5.47 (VSS_3), IC5.8 (VSSA), C10.1, C11.1, C12.1, C13.1, C14.1, C17.2, C17.2, C18.2, C18.2, C19.2, C19.2, C20.2, C25.2, C26.2, C27.2, C28.2, C29.2, C7.2, C8.1, C9.1, D3.2 (A), IC6.1 (VSS), IC7.2 (GND), IC8.6 (GND), IC8.9 (EP), J2.A1 (GND), J2.A12 (GND), J2.B1 (GND), J2.B12 (GND), J2.S1 (SHIELD), R12.2, R13.2, R35.1, R8.1, U1.7 (VSS), U3.29 (GND), U3.3 (GND), Y2.2 (GND_1), Y2.4 (GND_2)
- net VCC: now also C17.1, C19.1, D5.2 (A)
- net +3.3V: now reaches IC5.1 (VBAT)
- net +3.3V: now also IC5.24 (VDD_1), IC5.36 (VDD_2), IC5.48 (VDD_3), IC5.9 (VDDA), C19.1, C26.1, C27.1, C28.1, C29.1, IC7.5 (OUT), R11.2
- net OLED_SCL: now reaches IC5.21 (PB10)
- net OLED_SCL: now also R5.2, U1.10 (SCL)
- net OLED_SDA: now reaches IC5.22 (PB11)
- net OLED_SDA: now also R6.2, U1.11 (SDA)
- net MCU_CAN_RX: now reaches IC5.32 (PA11)
- net MCU_CAN_RX: now also U2.4 (R)
- net MCU_CAN_TX: now reaches IC5.33 (PA12)
- net MCU_CAN_TX: now also U2.1 (D)
- net OSC_IN: now reaches IC5.5 (PD0-OSC_IN)
- net OSC_IN: now also C7.1, Y2.1 (CRYSTAL_1)
- net OSC_OUT: now reaches IC5.6 (PD1-OSC_OUT)
- net OSC_OUT: now also C8.2, Y2.3 (CRYSTAL_2)
- net at IC5.7 (NRST): now also C25.1, R11.1
- new net: R8.2, U1.12 (IREF)
- new net: C15.1, U1.2 (c2n)
- new net: C15.2, U1.1 (c2p)
- new net: J2.A5 (CC1), R12.1
- new net: C13.2, C14.2, U1.14 (VCC)
- new net: C12.1, D3.1 (K), IC8.8 (PH), L1.1
- new net: C12.2, IC8.1 (BOOT)
- new net: D4.2 (A), J2.A4 (VBUS), J2.A9 (VBUS), J2.B4 (VBUS), J2.B9 (VBUS)
- new net: D5.1 (K), IC8.7 (VIN)
- new net: C12.2, U1.13 (VCOMH)
- new net: C16.2, U1.3 (c1p)
- new net: C16.1, U1.4 (c1n)
- new net: C9.2, R7.2, U1.9 (RES#)
- new net: IC8.4 (VSENSE), R34.1, R35.2
- new net: J2.B5 (CC2), R13.1
- new net: R15.1, U3.9 (~{RST})
- new net: C18.1, IC7.4 (BYPASS)
- new net +5V: C17.1, C18.1, C20.1, D4.1 (K), IC6.3 (VIN), IC7.1 (IN), IC7.3 (ON/~{OFF}), L1.2, R15.2, R34.2, U3.7 (VREGIN), U3.8 (VBUS)
- new net USART1_RXD: U3.26 (TXD)
- new net USART1_TXD: U3.25 (RXD)
- new net USB_DN: J2.A7 (D-), J2.B7 (D-), U3.5 (D-)
- new net USB_DP: J2.A6 (D+), J2.B6 (D+), U3.4 (D+)
- new net VCC_OLED: C10.2, C11.2, IC6.2 (VOUT), R5.1, R6.1, R7.1, U1.5 (VBAT), U1.8 (VDD)
- no-connect marks 3 -> 37
Other:
- note added: "MCU_Core"
- note added: "Motor_Driver Current Senser"
- note added: "OLED_Display"
- note added: "Power_Supply"
- note added: "USB_USART"
- moved on the sheet: C1, C2, C3, C4, C5, C6, D1, D2, IC1, IC2, IC3, IC4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

Commit message: Updata SCH Alpha0.3
Parts:
- removed C6: 220uF, symbol Device:C_Polarized
- removed D2: SS54, DIOM5126X245N, symbol SamacSys_Parts:SS54
- removed IC6: XC6206P332MR, SOT95P240X115-3N, symbol oled:XC6206P332MR
- removed J1: DC_IN, symbol Connector:Conn_01x02_Socket
- added C15, C19: 1uF, Capacitor_SMD:C_0603_1608Metric, symbol Device:C
- added C20: 0.01uF, Capacitor_SMD:C_0603_1608Metric, symbol Device:C
- added C29: 220uF, symbol Device:C_Polarized
- added C31: 0.1uF, Capacitor_SMD:C_0603_1608Metric, symbol Device:C
- added D4: SS54, DIOM5126X245N, symbol SamacSys_Parts:SS54
- added IC4: LP2992IM5-3.3, SOT95P280X145-5N, symbol SamacSys_Parts:LP2992IM5-3.3
- added J1: HALL_Sensor_Port, Connector_JST:JST_GH_SM05B-GHS-TB_1x05-1MP_P1.25mm_Horizontal, symbol Connector:Conn_01x05_Socket
- added J2: CAN_BUS_Port_IN, Connector_JST:JST_GH_BM02B-GHS-TBT_1x02-1MP_P1.25mm_Vertical, symbol Connector:Conn_01x02_Socket
- added J3: AS5600_Port, Connector_JST:JST_GH_BM04B-GHS-TBT_1x04-1MP_P1.25mm_Vertical, symbol Connector:Conn_01x04_Socket
- added J5: CAN_BUS_Port_OUT, Connector_JST:JST_GH_BM02B-GHS-TBT_1x02-1MP_P1.25mm_Vertical, symbol Connector:Conn_01x02_Socket
- added J6: DC_IN, Connector_AMASS:AMASS_XT30PW-M_1x02_P2.50mm_Horizontal, symbol Connector:Conn_01x02_Socket
- added J7: DC_OUT, Connector_AMASS:AMASS_XT30PW-M_1x02_P2.50mm_Horizontal, symbol Connector:Conn_01x02_Socket
- added J8: Conn_01x03_Socket, Connector_AMASS:AMASS_MR30PW-M_1x03_P3.50mm_Horizontal, symbol Connector:Conn_01x03_Socket
- added R10, R8: 4.7K, Resistor_SMD:R_0603_1608Metric, symbol oled:R
- added R17: 120R, Resistor_SMD:R_0603_1608Metric, symbol Device:R
- added R18: 0R, Resistor_SMD:R_0603_1608Metric, symbol Device:R
- C1: renamed from C25; footprint (none) -> Capacitor_SMD:C_0603_1608Metric
- C10: renamed from C26; footprint (none) -> Capacitor_SMD:C_0603_1608Metric
- C11: renamed from C27; footprint (none) -> Capacitor_SMD:C_0603_1608Metric
- C13: renamed from C28; footprint (none) -> Capacitor_SMD:C_0603_1608Metric
- C16: renamed from C8; value C -> 47pF; footprint (none) -> Capacitor_SMD:C_0603_1608Metric
- C2: renamed from C17; footprint (none) -> Capacitor_SMD:C_0603_1608Metric
- C3: renamed from C4; value C -> 47pF; footprint (none) -> Capacitor_SMD:C_0603_1608Metric
- C30: renamed from C3; footprint (none) -> Capacitor_SMD:C_0603_1608Metric
- C32: renamed from C1; footprint (none) -> Capacitor_SMD:C_0603_1608Metric
- C33: renamed from C2; footprint (none) -> Capacitor_SMD:C_0603_1608Metric
- C4: renamed from C5; value C -> 47pf; footprint (none) -> Capacitor_SMD:C_0603_1608Metric
- C6: renamed from C7; value C -> 47pF; footprint (none) -> Capacitor_SMD:C_0603_1608Metric
- C7: renamed from C19; footprint (none) -> Capacitor_SMD:C_0603_1608Metric
- C8: renamed from C18; footprint (none) -> Capacitor_SMD:C_0603_1608Metric
- C9: renamed from C29; footprint (none) -> Capacitor_SMD:C_0603_1608Metric
- D5: renamed from D1; footprint (none) -> LED_SMD:LED_0603_1608Metric
- J4: renamed from J2; footprint (none) -> Connector_USB:USB_C_Receptacle_XKB_U262-16XN-4BVC11
- R1: renamed from R11; footprint (none) -> Resistor_SMD:R_0603_1608Metric
- R11: renamed from R12; footprint (none) -> Resistor_SMD:R_0603_1608Metric
- R12: renamed from R13; footprint (none) -> Resistor_SMD:R_0603_1608Metric
- R13: renamed from R1; footprint (none) -> Resistor_SMD:R_0603_1608Metric
- R14: renamed from R2; footprint (none) -> Resistor_SMD:R_1206_3216Metric
- R15: renamed from R3; footprint (none) -> Resistor_SMD:R_1206_3216Metric
- R16: renamed from R4; footprint (none) -> Resistor_SMD:R_1206_3216Metric
- R4: renamed from R15; footprint (none) -> Resistor_SMD:R_0603_1608Metric
- renumbered C9 to C21, C10 to C22, C11 to C23, C12 to C24, C13 to C25, C14 to C26, C15 to C27, C16 to C28, D5 to D1, D3 to D2, D4 to D3, IC7 to IC1, IC5 to IC2, IC8 to IC3, IC2 to IC5, IC3 to IC6, IC4 to IC7, IC1 to IC8, R8 to R9, U3 to U1, U1 to U2, U2 to U3
Connections:
- net +3.3V: now also C22.2, C23.2, R7.1, U2.5 (VBAT), U2.8 (VDD), U3.3 (VCC), C31.2, R10.1, R8.1
- net +5V: now also C15.1, IC4.1 (IN), IC4.3 (ON/~{OFF})
- net GND: now also U3.2 (GND), C15.2, C19.2, C20.2, C29.2, C31.1, D4.2 (A), IC4.2 (GND), J1.5 (Pin_5), J3.4 (Pin_4), J6.1 (Pin_1), J7.1 (Pin_1)
- net ISense_U: now also IC2.12 (PA2); no longer IC2.10 (PA0-WKUP)
- net ISense_W: now also IC2.10 (PA0-WKUP); no longer IC2.12 (PA2)
- net Motor0_U: now also J8.3 (Pin_3)
- net Motor0_V: now also J8.2 (Pin_2)
- net Motor0_W: now also J8.1 (Pin_1)
- net OLED_SCL: now also IC2.45 (PB8); no longer IC2.21 (PB10)
- net OLED_SDA: now also IC2.46 (PB9); no longer IC2.22 (PB11)
- net USART1_RXD: now also IC2.43 (PB7)
- net USART1_TXD: now also IC2.42 (PB6)
- net VCC: now also C29.1, D4.1 (K), J6.2 (Pin_2), J7.2 (Pin_2)
- net VCC_OLED: no longer C22.2, C23.2, R7.1, U2.5 (VBAT), U2.8 (VDD)
- net CAN_DN: now reaches U3.6 (CANL)
- net CAN_DN: now also J2.2 (Pin_2), J5.2 (Pin_2), R18.1
- net CAN_DP: now reaches U3.7 (CANH)
- net CAN_DP: now also J2.1 (Pin_1), J5.1 (Pin_1), R17.2
- net MCU_CAN_RX renamed MCU_CAN_DN
- net MCU_CAN_TX renamed MCU_CAN_DP
- new net: R17.1, R18.2
- new net: C20.1, IC4.4 (BYPASS)
- new net AS5600_SCL: J3.2 (Pin_2), R8.2
- new net AS5600_SDA: J3.3 (Pin_3), R10.2
- new net HALL_A: J1.2 (Pin_2)
- new net HALL_B: J1.3 (Pin_3)
- new net HALL_C: J1.4 (Pin_4)
- new net VCC_Sensor: C19.1, IC4.5 (OUT), J1.1 (Pin_1), J3.1 (Pin_1)
Other:
- note added: "CAN_Transmiter"
- moved on the sheet: C12, C17, C18, C19, C20, D1, D2, IC3, L1, R34, R35, U3
